File: Headlights/Headlights.kicad_pcb (KiCad board)
At the start: 4 copper layers, 152.4 x 8.6 mm, 15 parts, among them Q1 Q_NMOS_GSD, Q2 Q_NPN_BCE

Commit message: ...
Routing:
- net VS: track 101.0 -> 1.21 mm
- net /PWM: track 16.3 -> 2.09 mm
- net Net-(Q1-Pad2): track 21.5 -> 7.99 mm
- removed copper zone on In1.Cu, net GNDREF
- removed copper zone on In2.Cu, net Net-(Q2-Pad2)
Changed lines of the file:
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@@
   (via (at 54.864 82.296) (size 0.45) (drill 0.2) (layers "F.Cu" "B.Cu") (free) (net 4))
   (via (at 56.388 84.328) (size 0.45) (drill 0.2) (layers "F.Cu" "B.Cu") (free) (net 4))
-  (segment (start 56.896 77.724) (end 56.388 78.232) (width 0.635) (layer "In2.Cu") (net 4))
-  (segment (start 155.702 78.486) (end 154.94 77.724) (width 0.635) (layer "In2.Cu") (net 4))
-  (segment (start 154.94 77.724) (end 56.896 77.724) (width 0.635) (layer "In2.Cu") (net 4))
   (segment (start 156.909 78.486) (end 155.702 78.486) (width 0.254) (layer "B.Cu") (net 4))
   (via (at 191.008 83.566) (size 0.45) (drill 0.2) (layers "F.Cu" "B.Cu") (free) (net 12))
@@
   (via (at 166.624 77.978) (size 0.45) (drill 0.2) (layers "F.Cu" "B.Cu") (net 13))
   (via (at 153.162 78.74) (size 0.45) (drill 0.2) (layers "F.Cu" "B.Cu") (net 13))
-  (segment (start 158.75 77.978) (end 166.624 77.978) (width 0.254) (layer "In2.Cu") (net 13))
-  (segment (start 153.67 79.248) (end 157.48 79.248) (width 0.254) (layer "In2.Cu") (net 13))
-  (segment (start 157.48 79.248) (end 158.75 77.978) (width 0.254) (layer "In2.Cu") (net 13))
-  (segment (start 153.162 78.74) (end 153.67 79.248) (width 0.254) (layer "In2.Cu") (net 13))
   (segment (start 166.944 78.298) (end 166.624 77.978) (width 0.254) (layer "B.Cu") (net 13))
   (segment (start 168.5775 78.298) (end 166.944 78.298) (width 0.254) (layer "B.Cu") (net 13))
   (via (at 183.89 79) (size 0.45) (drill 0.2) (layers "F.Cu" "B.Cu") (net 14))
   (via (at 170.434 78.74) (size 0.45) (drill 0.2) (layers "F.Cu" "B.Cu") (net 14))
-  (segment (start 183.642 78.74) (end 183.89 78.988) (width 0.254) (layer "In2.Cu") (net 14))
   (segment (start 183.89 78.988) (end 183.89 79) (width 0.254) (layer "In2.Cu") (net 14))
-  (segment (start 170.434 78.74) (end 183.642 78.74) (width 0.254) (layer "In2.Cu") (net 14))
   (segment (start 183.89 79) (end 182 79) (width 0.254) (layer "B.Cu") (net 14))
   (segment (start 169.611 80.198) (end 168.5775 80.198) (width 0.254) (layer "B.Cu") (net 14))
@@
       )
     )
-  )
-  (zone (net 2) (net_name "GNDREF") (layer "In1.Cu") (hatch edge 0.508)
-    (connect_pads (clearance 0.254))
-    (min_thickness 0.254) (filled_areas_thickness no)
-    (fill yes (thermal_gap 0.508) (thermal_bridge_width 0.508))
-    (polygon
-      (pts
-        (xy 203.2 85.598)
-        (xy 159.766 85.598)
-        (xy 159.766 76.962)
-        (xy 203.2 76.962)
-      )
-    )
-  )
-  (zone (net 12) (net_name "Net-(Q2-Pad2)") (layer "In2.Cu") (hatch edge 0.508)
-    (connect_pads (clearance 0.254))
-    (min_thickness 0.254) (filled_areas_thickness no)
-    (fill yes (thermal_gap 0.508) (thermal_bridge_width 0.508))
-    (polygon
-      (pts
-        (xy 201.676 83.058)
-        (xy 193.04 83.058)
-        (xy 193.04 85.598)
-        (xy 190.5 85.598)
-        (xy 190.5 76.962)
-        (xy 193.04 76.962)
-        (xy 193.04 79.502)
-        (xy 201.676 79.502)
-      )
-    )
